File: Final_Schematic (Eagle_design)/arduino_board_2iter.sch (EAGLE design)
At the start: 25 parts, among them IC1 LF356N

Commit message: PCB Updates as of 8/4/22
Parts:
- added PAD1, PAD2, PAD3: (no value), wirepad:1,6/0,9
Other:
- moved on the sheet: PD, TTL-1, TTL-2
Changed lines of the file:
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@@
 <part name="IC1" library="linear" deviceset="LF356" device="N"/>
 <part name="---15V" library="holes" deviceset="MOUNT-PAD-SQUARE" device="2.8"/>
+<part name="PAD1" library="wirepad" library_urn="urn:adsk.eagle:library:412" deviceset="1,6/0,9" device="" package3d_urn="urn:adsk.eagle:package:30840/1"/>
+<part name="PAD2" library="wirepad" library_urn="urn:adsk.eagle:library:412" deviceset="1,6/0,9" device="" package3d_urn="urn:adsk.eagle:package:30840/1"/>
+<part name="PAD3" library="wirepad" library_urn="urn:adsk.eagle:library:412" deviceset="1,6/0,9" device="" package3d_urn="urn:adsk.eagle:package:30840/1"/>
 </parts>
 <sheets>
@@
 <attribute name="VALUE" x="165.481" y="146.05" size="1.778" layer="96" rot="R90"/>
 </instance>
-<instance part="PD" gate="G$1" x="63.5" y="144.78" smashed="yes">
-<attribute name="NAME" x="58.41488125" y="150.500759375" size="1.42383125" layer="95"/>
-</instance>
-<instance part="TTL-1" gate="G$1" x="63.5" y="121.92" smashed="yes">
-<attribute name="NAME" x="58.41488125" y="127.640759375" size="1.42383125" layer="95"/>
-</instance>
-<instance part="TTL-2" gate="G$1" x="63.5" y="99.06" smashed="yes">
-<attribute name="NAME" x="58.41488125" y="104.780759375" size="1.42383125" layer="95"/>
+<instance part="PD" gate="G$1" x="63.5" y="144.78" smashed="yes" rot="MR0">
+<attribute name="NAME" x="68.58511875" y="150.500759375" size="1.42383125" layer="95" rot="MR0"/>
+</instance>
+<instance part="TTL-1" gate="G$1" x="63.5" y="121.92" smashed="yes" rot="MR0">
+<attribute name="NAME" x="68.58511875" y="127.640759375" size="1.42383125" layer="95" rot="MR0"/>
+</instance>
+<instance part="TTL-2" gate="G$1" x="63.5" y="99.06" smashed="yes" rot="MR0">
+<attribute name="NAME" x="68.58511875" y="104.780759375" size="1.42383125" layer="95" rot="MR0"/>
 </instance>
 <instance part="FILTER" gate="G$1" x="231.14" y="127" smashed="yes" rot="R90">
@@
 <instance part="---15V" gate="G$1" x="162.56" y="180.34" smashed="yes" rot="R180">
 <attribute name="NAME" x="159.766" y="179.7558" size="1.778" layer="95" rot="R180"/>
+</instance>
+<instance part="PAD1" gate="1" x="40.64" y="152.4" smashed="yes">
+<attribute name="NAME" x="39.497" y="154.2542" size="1.778" layer="95"/>
+<attribute name="VALUE" x="39.497" y="149.098" size="1.778" layer="96"/>
+</instance>
+<instance part="PAD2" gate="1" x="40.64" y="147.32" smashed="yes">
+<attribute name="NAME" x="39.497" y="149.1742" size="1.778" layer="95"/>
+<attribute name="VALUE" x="39.497" y="144.018" size="1.778" layer="96"/>
+</instance>
+<instance part="PAD3" gate="1" x="40.64" y="142.24" smashed="yes">
+<attribute name="NAME" x="39.497" y="144.0942" size="1.778" layer="95"/>
+<attribute name="VALUE" x="39.497" y="138.938" size="1.778" layer="96"/>
 </instance>
 </instances>
@@
 <pinref part="TTL-2" gate="G$1" pin="2"/>
 <pinref part="TTL-2" gate="G$1" pin="SHIELD"/>
-<wire x1="71.12" y1="99.06" x2="71.12" y2="93.98" width="0.1524" layer="91"/>
-<wire x1="71.12" y1="93.98" x2="50.8" y2="93.98" width="0.1524" layer="91"/>
-<junction x="71.12" y="93.98"/>
+<wire x1="55.88" y1="99.06" x2="55.88" y2="93.98" width="0.1524" layer="91"/>
+<wire x1="55.88" y1="93.98" x2="50.8" y2="93.98" width="0.1524" layer="91"/>
+<junction x="55.88" y="93.98"/>
 <pinref part="TTL-1" gate="G$1" pin="2"/>
 <pinref part="TTL-1" gate="G$1" pin="SHIELD"/>
-<wire x1="71.12" y1="121.92" x2="71.12" y2="116.84" width="0.1524" layer="91"/>
+<wire x1="55.88" y1="121.92" x2="55.88" y2="116.84" width="0.1524" layer="91"/>
 <wire x1="50.8" y1="93.98" x2="50.8" y2="116.84" width="0.1524" layer="91"/>
-<wire x1="50.8" y1="116.84" x2="71.12" y2="116.84" width="0.1524" layer="91"/>
-<junction x="71.12" y="116.84"/>
+<wire x1="50.8" y1="116.84" x2="55.88" y2="116.84" width="0.1524" layer="91"/>
+<junction x="55.88" y="116.84"/>
 <pinref part="PD" gate="G$1" pin="2"/>
 <pinref part="PD" gate="G$1" pin="SHIELD"/>
-<wire x1="71.12" y1="144.78" x2="71.12" y2="139.7" width="0.1524" layer="91"/>
+<wire x1="55.88" y1="144.78" x2="55.88" y2="139.7" width="0.1524" layer="91"/>
 <wire x1="50.8" y1="116.84" x2="50.8" y2="139.7" width="0.1524" layer="91"/>
-<wire x1="50.8" y1="139.7" x2="71.12" y2="139.7" width="0.1524" layer="91"/>
+<wire x1="50.8" y1="139.7" x2="55.88" y2="139.7" width="0.1524" layer="91"/>
 <junction x="50.8" y="116.84"/>
-<junction x="71.12" y="139.7"/>
+<junction x="55.88" y="139.7"/>
 <wire x1="50.8" y1="139.7" x2="50.8" y2="170.18" width="0.1524" layer="91"/>
 <wire x1="50.8" y1="170.18" x2="93.98" y2="170.18" width="0.1524" layer="91"/>
@@
 <wire x1="241.3" y1="142.24" x2="241.3" y2="127" width="0.1524" layer="91"/>
 <wire x1="241.3" y1="127" x2="241.3" y2="119.38" width="0.1524" layer="91"/>
-<wire x1="71.12" y1="93.98" x2="88.9" y2="93.98" width="0.1524" layer="91"/>
+<wire x1="55.88" y1="93.98" x2="88.9" y2="93.98" width="0.1524" layer="91"/>
 <pinref part="LLC" gate="G$1" pin="GND"/>
 <wire x1="88.9" y1="93.98" x2="88.9" y2="60.96" width="0.1524" layer="91"/>
@@
 <segment>
 <pinref part="TTL-1" gate="G$1" pin="1"/>
-<wire x1="71.12" y1="124.46" x2="73.66" y2="124.46" width="0.1524" layer="91"/>
+<wire x1="55.88" y1="124.46" x2="73.66" y2="124.46" width="0.1524" layer="91"/>
 <wire x1="73.66" y1="124.46" x2="73.66" y2="73.66" width="0.1524" layer="91"/>
 <pinref part="LLC" gate="G$1" pin="HV1"/>
@@
 <segment>
 <pinref part="TTL-2" gate="G$1" pin="1"/>
-<wire x1="71.12" y1="101.6" x2="76.2" y2="101.6" width="0.1524" layer="91"/>
+<wire x1="55.88" y1="101.6" x2="76.2" y2="101.6" width="0.1524" layer="91"/>
 <pinref part="LLC" gate="G$1" pin="HV2"/>
 <wire x1="76.2" y1="101.6" x2="76.2" y2="71.12" width="0.1524" layer="91"/>
@@
 <segment>
 <pinref part="PD" gate="G$1" pin="1"/>
-<wire x1="71.12" y1="147.32" x2="81.28" y2="147.32" width="0.1524" layer="91"/>
+<wire x1="55.88" y1="147.32" x2="81.28" y2="147.32" width="0.1524" layer="91"/>
 <wire x1="81.28" y1="147.32" x2="81.28" y2="55.88" width="0.1524" layer="91"/>
 <wire x1="81.28" y1="55.88" x2="88.9" y2="55.88" width="0.1524" layer="91"/>
@@
 </schematic>
 </drawing>
+<compatibility>
+<note version="8.2" severity="warning">
+Since Version 8.2, EAGLE supports online libraries. The ids
+of those online libraries will not be understood (or retained)
+with this version.
+</note>
+<note version="8.3" severity="warning">
+Since Version 8.3, EAGLE supports URNs for individual library
+assets (packages, symbols, and devices). The URNs of those assets
+will not be understood (or retained) with this version.
+</note>
+<note version="8.3" severity="warning">
+Since Version 8.3, EAGLE supports the association of 3D packages
+with devices in libraries, schematics, and board files. Those 3D
+packages will not be understood (or retained) with this version.
+</note>
+</compatibility>
 </eagle>

Commit message: PCB Updates as of 8/9/22
Parts:
- added PAD4, PAD5: (no value), wirepad:1,6/0,9
Changed lines of the file:
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@@
 <part name="PAD2" library="wirepad" library_urn="urn:adsk.eagle:library:412" deviceset="1,6/0,9" device="" package3d_urn="urn:adsk.eagle:package:30840/1"/>
 <part name="PAD3" library="wirepad" library_urn="urn:adsk.eagle:library:412" deviceset="1,6/0,9" device="" package3d_urn="urn:adsk.eagle:package:30840/1"/>
+<part name="PAD4" library="wirepad" library_urn="urn:adsk.eagle:library:412" deviceset="1,6/0,9" device="" package3d_urn="urn:adsk.eagle:package:30840/1"/>
+<part name="PAD5" library="wirepad" library_urn="urn:adsk.eagle:library:412" deviceset="1,6/0,9" device="" package3d_urn="urn:adsk.eagle:package:30840/1"/>
 </parts>
 <sheets>
@@
 <attribute name="VALUE" x="39.497" y="138.938" size="1.778" layer="96"/>
 </instance>
+<instance part="PAD4" gate="1" x="40.64" y="137.16" smashed="yes">
+<attribute name="NAME" x="39.497" y="139.0142" size="1.778" layer="95"/>
+<attribute name="VALUE" x="39.497" y="133.858" size="1.778" layer="96"/>
+</instance>
+<instance part="PAD5" gate="1" x="40.64" y="132.08" smashed="yes">
+<attribute name="NAME" x="39.497" y="133.9342" size="1.778" layer="95"/>
+<attribute name="VALUE" x="39.497" y="128.778" size="1.778" layer="96"/>
+</instance>
 </instances>
